File: pcb/panel/wombus64_led.kicad_pcb (KiCad board)
At the start: 2 copper layers, 100 x 100 mm, 116 parts, among them J1 Conn_01x02_Pin, J2 Conn_01x02_Pin, J3 Conn_01x02_Pin, J4 Conn_01x02_Pin, J5 Conn_01x02_Pin, U1 AP62401WU, U3 SN74LVC1G125DCK

Commit message: added bill of materials
Parts:
- C1: value TBD -> 10μF
- C2, C3: value TBDuF -> 100uF
- C5: value TBD -> 100pF
- C6: value TBD -> 0.1μF
- D65: value B1911B -> B1911R
- R1: value 52.3Ω -> 52.3kΩ
Changed lines of the file:
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@@
 			)
 		)
-		(property "Value" "B1911B"
+		(property "Value" "B1911R"
 			(at 0 -1.43 90)
 			(layer "B.Fab")
@@
 			)
 		)
-		(property "Value" "TBDuF"
+		(property "Value" "100uF"
 			(at 2.5 -5.25 0)
 			(layer "B.Fab")
@@
 			)
 		)
-		(property "Value" "TBDuF"
+		(property "Value" "100uF"
 			(at 2.5 -5.25 0)
 			(layer "B.Fab")
@@
 			)
 		)
-		(property "Value" "TBD"
+		(property "Value" "0.1μF"
 			(at 0 -1.43 90)
 			(layer "B.Fab")
@@
 			)
 		)
-		(property "Value" "52.3Ω"
+		(property "Value" "52.3kΩ"
 			(at 0 -1.43 90)
 			(layer "B.Fab")
@@
 			)
 		)
-		(property "Value" "TBD"
+		(property "Value" "100pF"
 			(at 0 -1.43 90)
 			(layer "B.Fab")
@@
 			)
 		)
-		(property "Value" "TBD"
+		(property "Value" "10μF"
 			(at 0 -1.43 0)
 			(layer "B.Fab")
@@
 			(pts
 				(xy 152 87.5) (xy 153.75 85.5) (xy 154.75 84.5) (xy 149 84.5) (xy 150.75 86.25) (xy 150.75 87.5)
-				(xy 150.75 87.5)
 			)
 		)
