File: pcb/panel/wombus64_led.kicad_sch (KiCad schematic)
At the start: 116 parts, among them J1 Conn_01x02_Pin, J2 Conn_01x02_Pin, J3 Conn_01x02_Pin, J4 Conn_01x02_Pin, J5 Conn_01x02_Pin, U1 AP62401WU, U3 SN74LVC1G125DCK

Commit message: added bill of materials
Parts:
- C1: value TBD -> 10μF
- C2, C3: value TBDuF -> 100uF
- C5: value TBD -> 100pF
- C6: value TBD -> 0.1μF
- D65: value B1911B -> B1911R
- R1: value 52.3Ω -> 52.3kΩ
Changed lines of the file:
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@@
 			)
 		)
-		(property "Value" "TBD"
+		(property "Value" "0.1μF"
 			(at 330.2 91.948 0)
 			(effects
@@
 			)
 		)
-		(property "Value" "B1911B"
+		(property "Value" "B1911R"
 			(at 360.68 56.1974 90)
 			(effects
@@
 			)
 		)
-		(property "Value" "TBDuF"
+		(property "Value" "100uF"
 			(at 365.252 91.948 0)
 			(effects
@@
 			)
 		)
-		(property "Value" "TBDuF"
+		(property "Value" "100uF"
 			(at 357.632 91.948 0)
 			(effects
@@
 			)
 		)
-		(property "Value" "TBD"
-			(at 295.91 94.488 0)
+		(property "Value" "10μF"
+			(at 295.402 94.488 0)
 			(effects
 				(font
@@
 			)
 		)
-		(property "Value" "TBD"
-			(at 342.9 91.948 0)
+		(property "Value" "100pF"
+			(at 341.63 92.456 0)
 			(effects
 				(font
@@
 			)
 		)
-		(property "Value" "52.3Ω"
+		(property "Value" "52.3kΩ"
 			(at 348.488 88.646 90)
 			(effects
